File: hardware-FeatherS3/lg_hvac_esp32.kicad_pcb (KiCad board)
At the start: 4 copper layers, 22.9 x 50.8 mm, 19 parts, among them J1 JST_XH_S3B-XH-A-1_01x03, J2 Conn_01x16, J3 Conn_01x12, U1 TPS82130, U2 TJA1027

Commit message: New Rev.20260717, with added C3.
Context: https://github.com/JanM321/esphome-lg-controller/issues/156
Parts:
- added C3: C_0805_2012Metric, Capacitor_SMD:C_0805_2012Metric, F.Cu at (98.7, 54.4)
- moved R3 2.16 mm to (98.7, 52.3)
- moved R2 1.09 mm to (98.9, 49.5)
- moved R1 1.05 mm to (95.6, 49.5)
Routing:
- net +3V3: track 19.0 -> 21.5 mm
- net GND: track 12.3 -> 14.7 mm
- net Net-(U1-PG): track 4.97 -> 4.11 mm
- net Net-(U1-FB): track 8.08 -> 8.88 mm
Other:
- board text added: "LG HVAC ESP32 Controller Rev.20260717"
- board text removed: "LG HVAC ESP32 Controller Rev.20250519"
